Commit message: fix_urdf.xacro_and_launch_file_and_cmakelist

File: cvg_sim_gazebo/urdf/quadrotor_base.urdf.xacro (robot description, xacro)
@@ -6,5 +6,5 @@
 >
   <xacro:include filename="$(find cvg_sim_gazebo_plugins)/urdf/quadrotor_plugins.urdf.xacro" />
-  <property name="pi" value="3.1415926535897931" />
+  <xacro:property name="pi" value="3.1415926535897931" />
   <!-- Main quadrotor link -->
   <xacro:macro name="quadrotor_base_macro">

File: cvg_sim_gazebo/urdf/quadrotor_sensors.urdf.xacro (robot description, xacro)
@@ -5,5 +5,5 @@
 xmlns:interface="http://playerstage.sourceforge.net/gazebo/xmlschema/#interface"
 xmlns:xacro="http://playerstage.sourceforge.net/gazebo/xmlschema/#interface">
-    <property name="M_PI" value="3.1415926535897931" />
+    <xacro:property name="M_PI" value="3.1415926535897931" />
     <!-- Included URDF Files -->
     <xacro:include filename="$(find cvg_sim_gazebo)/urdf/quadrotor_base.urdf.xacro" />

File: cvg_sim_gazebo/urdf/sensors/generic_camera.urdf.xacro (robot description, xacro)
@@ -5,8 +5,8 @@
   xmlns:xacro="http://ros.org/wiki/xacro"
   >
-    <property name="M_PI" value="3.1415926535897931" />
+    <xacro:property name="M_PI" value="3.1415926535897931" />
     <xacro:macro name="generic_camera" params="name sim_name parent *origin update_rate res_x res_y image_format hfov">
       <joint name="${name}_joint" type="fixed">
-        <insert_block name="origin" />
+        <xacro:insert_block name="origin" />
         <parent link="${parent}"/>
         <child link="${name}_link"/>

File: cvg_sim_gazebo/urdf/sensors/hokuyo_utm30lx.urdf.xacro (robot description, xacro)
@@ -7,5 +7,5 @@
     <xacro:macro name="hokuyo_utm30lx" params="name parent *origin ros_topic update_rate ray_count min_angle max_angle">
       <joint name="${name}_joint" type="fixed">
-	<insert_block name="origin" />
+	<xacro:insert_block name="origin" />
 	<parent link="${parent}"/>
 	<child link="${name}_frame"/>
