Commit message: fix_hokuyo_lidar_pub

File: cvg_sim_gazebo/urdf/quadrotor_sensors.urdf.xacro (robot description, xacro)
@@ -15,18 +15,18 @@
       <origin xyz="-0.15 0.0 0.0" rpy="0 ${90*M_PI/180} 0"/>
     </xacro:sonar_sensor>
-    <!-- Hokuyo UTM-30LX mounted upside down below the quadrotor body
+    <!-- Hokuyo UTM-30LX mounted upside down below the quadrotor body -->
     <xacro:include filename="$(find cvg_sim_gazebo)/urdf/sensors/hokuyo_utm30lx.urdf.xacro" />
-    <xacro:hokuyo_utm30lx name="laser0" parent="base_link" ros_topic="scan" update_rate="40" ray_count="1081" min_angle="135" max_angle="-135">
+    <xacro:hokuyo_utm30lx name="laser0" parent="base_link" ros_topic="scan" update_rate="40" ray_count="1081" min_angle="${135*M_PI/180}" max_angle="${-135*M_PI/180}">
       <origin xyz="0.0 0.0 0.08" rpy="${M_PI} 0 0"/>
-    </xacro:hokuyo_utm30lx>-->
+    </xacro:hokuyo_utm30lx>
     <!-- The following two cameras should be united to one! -->
     <!-- Forward facing camera -->
     <xacro:include filename="$(find cvg_sim_gazebo)/urdf/sensors/generic_camera.urdf.xacro" />
-    <xacro:generic_camera name="front" sim_name="ardrone" parent="base_link" update_rate="60" res_x="640" res_y="360" image_format="R8G8B8" hfov="${81*M_PI/180}">
+    <xacro:generic_camera name="front" sim_name="ardrone" parent="base_link" update_rate="60" res_x="640" res_y="480" image_format="R8G8B8" hfov="${81*M_PI/180}">
       <origin xyz="0.21 0.0 0.01" rpy="0 0 0"/>
     </xacro:generic_camera>
     <!-- Downward facing camera -->
     <xacro:include filename="$(find cvg_sim_gazebo)/urdf/sensors/generic_camera.urdf.xacro" />
-    <xacro:generic_camera name="bottom" sim_name="ardrone" parent="base_link" update_rate="60" res_x="640" res_y="360" image_format="R8G8B8" hfov="${81*M_PI/180}">
+    <xacro:generic_camera name="bottom" sim_name="ardrone" parent="base_link" update_rate="60" res_x="640" res_y="480" image_format="R8G8B8" hfov="${81*M_PI/180}">
       <origin xyz="0.15 0.0 0.0" rpy="0 ${M_PI/2} 0"/>
     </xacro:generic_camera>

File: cvg_sim_gazebo/urdf/sensors/hokuyo_utm30lx.urdf.xacro (robot description, xacro)
@@ -11,46 +11,52 @@
 	<child link="${name}_frame"/>
       </joint>
-<link name="${name}_frame">
-	<inertial>
-	  <mass value="0.001" />
-	  <origin xyz="0 0 0" rpy="0 0 0" />
-		<inertia ixx="0.0001" ixy="0" ixz="0" iyy="0.0001" iyz="0" izz="0.0001" />
-	</inertial>
-	<visual>
-	  <origin xyz="0 0 0" rpy="0 0 0" />
-          <geometry>
-          <mesh filename="package://cvg_sim_gazebo/meshes/hokuyo_utm30lx/hokuyo_utm_30lx$(optenv TEST_SELF_FILTER).dae"/>
-        </geometry>
-	</visual>
-	<collision>
-	  <origin xyz="0 0 -0.0115" rpy="0 0 0" />
-          <geometry>
-          <box size="0.058 0.058 0.087" />
-          <!--<mesh filename="package://hector_sensors_description/meshes/hokuyo_utm30lx/hokuyo_utm_30lx.stl"/>-->
-        </geometry>
-	</collision>
-</link>
+	<link name="${name}_frame">
+		<inertial>
+			<mass value="0.001" />
+			<origin xyz="0 0 0" rpy="0 0 0" />
+			<inertia ixx="0.0001" ixy="0" ixz="0" iyy="0.0001" iyz="0" izz="0.0001" />
+		</inertial>
+		<visual>
+			<origin xyz="0 0 0" rpy="0 0 0" />
+		        <geometry>
+		        <mesh filename="package://cvg_sim_gazebo/meshes/hokuyo_utm30lx/hokuyo_utm_30lx$(optenv TEST_SELF_FILTER).dae"/>
+		      </geometry>
+		</visual>
+		<collision>
+			<origin xyz="0 0 -0.0115" rpy="0 0 0" />
+		        <geometry>
+		        <box size="0.058 0.058 0.087" />
+		       </geometry>
+		</collision>
+	</link>
   <gazebo reference="${name}_frame">
-    <sensor:ray name="${name}">
-    <rayCount>${ray_count}</rayCount>
-    <rangeCount>${ray_count}</rangeCount>
-        <laserCount>1</laserCount>
-        <origin>0.0 0.0 0.0</origin>
-        <displayRays>false</displayRays>
-        <minAngle>${min_angle}</minAngle>
-        <maxAngle>${max_angle}</maxAngle>
-        <minRange>0.08</minRange>
-        <maxRange>30.0</maxRange>
-        <resRange>0.01</resRange>
-        <updateRate>${update_rate}</updateRate>
-        <controller:gazebo_ros_laser name="gazebo_ros_${name}_controller" plugin="libgazebo_ros_laser.so">
-          <gaussianNoise>0.005</gaussianNoise>
-          <alwaysOn>true</alwaysOn>
-          <updateRate>${update_rate}</updateRate>
-          <topicName>${ros_topic}</topicName>
-          <frameName>${name}_frame</frameName>
-          <interface:laser name="gazebo_ros_${name}_iface" />
-        </controller:gazebo_ros_laser>
-      </sensor:ray>
+        <sensor type="ray" name="${name}">
+            <always_on>true</always_on>
+            <pose>0 0 0 0 0 0</pose>
+            <visualize>true</visualize>
+            <update_rate>${update_rate}</update_rate>
+            <ray>
+                <scan>
+                    <horizontal>
+                        <samples>${ray_count}</samples>
+                        <resolution>1</resolution>
+                        <min_angle>${min_angle}</min_angle>
+                        <max_angle>${max_angle}</max_angle>
+                    </horizontal>
+                </scan>
+                <range>
+                    <min>0.08</min>
+                    <max>30</max>
+                    <resolution>0.01</resolution>
+                </range>
+           </ray>
+	         <plugin name="gazebo_ros_${name}_controller" filename="libgazebo_ros_laser.so">
+	           <gaussianNoise>0.005</gaussianNoise>
+	           <alwaysOn>true</alwaysOn>
+	           <updateRate>${update_rate}</updateRate>
+	           <topicName>${ros_topic}</topicName>
+	           <frameName>${name}_frame</frameName>
+	         </plugin>
+        </sensor>
     </gazebo>
     </xacro:macro>

Commit message: fix_hokuyo_utm30lx_origin

File: cvg_sim_gazebo/urdf/quadrotor_sensors.urdf.xacro (robot description, xacro)
@@ -18,5 +18,5 @@
     <xacro:include filename="$(find cvg_sim_gazebo)/urdf/sensors/hokuyo_utm30lx.urdf.xacro" />
     <xacro:hokuyo_utm30lx name="laser0" parent="base_link" ros_topic="scan" update_rate="40" ray_count="1081" min_angle="${135*M_PI/180}" max_angle="${-135*M_PI/180}">
-      <origin xyz="0.0 0.0 0.08" rpy="${M_PI} 0 0"/>
+      <origin xyz="0.0 0.0 0.08" rpy="0 0 0"/>
     </xacro:hokuyo_utm30lx>
     <!-- The following two cameras should be united to one! -->

Commit message: add_gimbal_macro

File: cvg_sim_gazebo/urdf/quadrotor_sensors.urdf.xacro (robot description, xacro)
@@ -1,4 +1,4 @@
 <?xml version="1.0"?>
-<robot name="quadrotor_hokuyo_utm30lx"
+<robot name="quadrotor_sensors"
 xmlns:sensor="http://playerstage.sourceforge.net/gazebo/xmlschema/#sensor"
 xmlns:controller="http://playerstage.sourceforge.net/gazebo/xmlschema/#controller"
@@ -10,4 +10,8 @@
     <!-- Instantiate quadrotor_base_macro once (has no parameters atm) -->
     <quadrotor_base_macro />
+    <!-- Gimbal  -->
+    <xacro:gimbal_macro namespace="${namespace}">
+      <origin xyz="0 0 0" rpy="0 0 0" />
+    </xacro:gimbal_macro>
     <!-- Sonar height sensor -->
     <xacro:include filename="$(find cvg_sim_gazebo)/urdf/sensors/sonar_sensor.urdf.xacro" />
